Commit message: Add files via upload

File: src/rover/urdf/rover.urdf.xacro (robot description, xacro)
@@ -1,16 +1,29 @@
 <?xml version="1.0"?>
 <robot xmlns:xacro="http://www.ros.org/wiki/xacro" name="rover">
-  <!-- ================= Constants ================= -->
-  <xacro:property name="base_length"  value="1.5"/>
-  <xacro:property name="base_width"   value="2.0"/>
+  <!-- ===================== Constants ===================== -->
+  <!-- Bikin sisi panjang mengikuti sumbu X (maju) -->
+  <xacro:property name="base_length"  value="2.0"/>   <!-- arah X -->
+  <xacro:property name="base_width"   value="1.5"/>   <!-- arah Y -->
   <xacro:property name="base_height"  value="0.8"/>
   <xacro:property name="wheel_radius" value="0.133"/>
   <xacro:property name="wheel_width"  value="0.3"/>
-  <!-- Z offset of wheel centre above base_link frame -->
+  <!-- Z posisi pusat roda terhadap frame base_link (z=0 di lantai) -->
   <xacro:property name="wheel_origin_z" value="${wheel_radius}"/>
-  <!-- ================= Base Link ================= -->
+  <!-- Offset roda dari ujung-ujung base (biar tidak mepet) -->
+  <xacro:property name="edge_margin_x" value="0.10"/>
+  <xacro:property name="wheel_x" value="${base_length/2 - edge_margin_x}"/>
+  <!-- Posisikan roda di luar sisi base (tambah setengah lebar roda) -->
+  <xacro:property name="wheel_y" value="${base_width/2 + wheel_width/2}"/>
+  <!-- ===================== Frames (opsional tapi rapi) ===================== -->
+  <link name="base_footprint"/>
+  <joint name="base_footprint_to_base_link" type="fixed">
+    <parent link="base_footprint"/>
+    <child  link="base_link"/>
+    <origin xyz="0 0 0" rpy="0 0 0"/>
+  </joint>
+  <!-- ===================== Base Link ===================== -->
   <link name="base_link">
     <visual>
-      <!-- Place the box so its bottom rests on z=0 -->
+      <!-- Letakkan box sehingga sisi bawah pas di z=0 -->
       <origin xyz="0 0 ${base_height/2}" rpy="0 0 0"/>
       <geometry>
@@ -21,11 +34,18 @@
       </material>
     </visual>
+    <!-- (opsional) collision sama dengan visual -->
+    <collision>
+      <origin xyz="0 0 ${base_height/2}" rpy="0 0 0"/>
+      <geometry>
+        <box size="${base_length} ${base_width} ${base_height}"/>
+      </geometry>
+    </collision>
   </link>
-  <!-- ================= Wheel Macro ================= -->
+  <!-- ===================== Wheel Macro ===================== -->
   <xacro:macro name="wheel" params="name parent x y">
     <link name="${name}">
       <visual>
-        <!-- Rotate cylinder so its axis points along y -->
-        <origin xyz="0 0 0" rpy="0 1.5708 0"/>
+        <!-- Putar silinder 90° di sumbu X supaya sumbu silinder = Y (sumbu putar roda) -->
+        <origin xyz="0 0 0" rpy="1.5708 0 0"/>
         <geometry>
           <cylinder radius="${wheel_radius}" length="${wheel_width}"/>
@@ -35,4 +55,10 @@
         </material>
       </visual>
+      <collision>
+        <origin xyz="0 0 0" rpy="1.5708 0 0"/>
+        <geometry>
+          <cylinder radius="${wheel_radius}" length="${wheel_width}"/>
+        </geometry>
+      </collision>
     </link>
     <joint name="joint_${name}" type="fixed">
@@ -42,8 +68,9 @@
     </joint>
   </xacro:macro>
-  <!-- ================= Instantiate Wheels ================= -->
-  <xacro:wheel name="wheel_front_left"  parent="base_link" x=" 0.90" y=" 0.873"/>
-  <xacro:wheel name="wheel_front_right" parent="base_link" x=" 0.90" y="-0.873"/>
-  <xacro:wheel name="wheel_rear_left"   parent="base_link" x="-0.90" y=" 0.873"/>
-  <xacro:wheel name="wheel_rear_right"  parent="base_link" x="-0.90" y="-0.873"/>
+  <!-- ===================== Instantiate 4 Wheels ===================== -->
+  <!-- Depan = +X, Kiri = +Y -->
+  <xacro:wheel name="wheel_front_left"  parent="base_link" x="${ wheel_x}" y="${ wheel_y}"/>
+  <xacro:wheel name="wheel_front_right" parent="base_link" x="${ wheel_x}" y="${-wheel_y}"/>
+  <xacro:wheel name="wheel_rear_left"   parent="base_link" x="${-wheel_x}" y="${ wheel_y}"/>
+  <xacro:wheel name="wheel_rear_right"  parent="base_link" x="${-wheel_x}" y="${-wheel_y}"/>
 </robot>

Commit message: Add files via upload

File: src/rover/urdf/rover.urdf.xacro (robot description, xacro)
@@ -1,76 +1,86 @@
 <?xml version="1.0"?>
-<robot xmlns:xacro="http://www.ros.org/wiki/xacro" name="rover">
-  <!-- ===================== Constants ===================== -->
-  <!-- Bikin sisi panjang mengikuti sumbu X (maju) -->
-  <xacro:property name="base_length"  value="2.0"/>   <!-- arah X -->
-  <xacro:property name="base_width"   value="1.5"/>   <!-- arah Y -->
-  <xacro:property name="base_height"  value="0.8"/>
-  <xacro:property name="wheel_radius" value="0.133"/>
-  <xacro:property name="wheel_width"  value="0.3"/>
-  <!-- Z posisi pusat roda terhadap frame base_link (z=0 di lantai) -->
-  <xacro:property name="wheel_origin_z" value="${wheel_radius}"/>
-  <!-- Offset roda dari ujung-ujung base (biar tidak mepet) -->
-  <xacro:property name="edge_margin_x" value="0.10"/>
-  <xacro:property name="wheel_x" value="${base_length/2 - edge_margin_x}"/>
-  <!-- Posisikan roda di luar sisi base (tambah setengah lebar roda) -->
-  <xacro:property name="wheel_y" value="${base_width/2 + wheel_width/2}"/>
-  <!-- ===================== Frames (opsional tapi rapi) ===================== -->
-  <link name="base_footprint"/>
-  <joint name="base_footprint_to_base_link" type="fixed">
-    <parent link="base_footprint"/>
-    <child  link="base_link"/>
-    <origin xyz="0 0 0" rpy="0 0 0"/>
-  </joint>
-  <!-- ===================== Base Link ===================== -->
+<robot xmlns:xacro="http://www.ros.org/wiki/xacro" name="rover_rigid_y_wheels">
+  <!-- materials -->
+  <material name="gray"><color rgba="0.7 0.7 0.7 1.0"/></material>
+  <material name="black"><color rgba="0.1 0.1 0.1 1.0"/></material>
+  <material name="dark"><color rgba="0.2 0.2 0.25 1.0"/></material>
+  <material name="red"><color rgba="0.8 0.1 0.1 1.0"/></material>
+  <material name="silver"><color rgba="0.8 0.8 0.9 1.0"/></material>
+  <!-- Constants -->
+  <xacro:property name="base_length" value="1.0"/>
+  <xacro:property name="base_width" value="0.5"/>
+  <xacro:property name="base_height" value="0.25"/>
+  <xacro:property name="arm_length" value="0.6"/>
+  <xacro:property name="arm_thickness" value="0.08"/>
+  <xacro:property name="arm_depth" value="0.06"/>
+  <xacro:property name="wheel_radius" value="0.165"/>
+  <xacro:property name="wheel_width" value="0.3"/>
+  <!-- BASE LINK -->
   <link name="base_link">
     <visual>
-      <!-- Letakkan box sehingga sisi bawah pas di z=0 -->
-      <origin xyz="0 0 ${base_height/2}" rpy="0 0 0"/>
-      <geometry>
-        <box size="${base_length} ${base_width} ${base_height}"/>
-      </geometry>
-      <material name="gray">
-        <color rgba="0.7 0.7 0.7 1.0"/>
-      </material>
+      <origin xyz="0 0 0" rpy="0 0 0"/>
+      <geometry><box size="${base_length} ${base_width} ${base_height}"/></geometry>
+      <material name="red"/>
     </visual>
-    <!-- (opsional) collision sama dengan visual -->
     <collision>
-      <origin xyz="0 0 ${base_height/2}" rpy="0 0 0"/>
-      <geometry>
-        <box size="${base_length} ${base_width} ${base_height}"/>
-      </geometry>
+      <origin xyz="0 0 0" rpy="0 0 0"/>
+      <geometry><box size="${base_length} ${base_width} ${base_height}"/></geometry>
     </collision>
   </link>
-  <!-- ===================== Wheel Macro ===================== -->
-  <xacro:macro name="wheel" params="name parent x y">
+  <!-- ARM MACRO -->
+  <xacro:macro name="arm" params="name parent x_pos y_pos visual_origin visual_rpy">
     <link name="${name}">
       <visual>
-        <!-- Putar silinder 90° di sumbu X supaya sumbu silinder = Y (sumbu putar roda) -->
-        <origin xyz="0 0 0" rpy="1.5708 0 0"/>
-        <geometry>
-          <cylinder radius="${wheel_radius}" length="${wheel_width}"/>
-        </geometry>
-        <material name="black">
-          <color rgba="0.1 0.1 0.1 1.0"/>
-        </material>
+        <origin xyz="${visual_origin}" rpy="${visual_rpy}"/>
+        <geometry><box size="${arm_length} ${arm_thickness} ${arm_depth}"/></geometry>
+        <material name="silver"/>
       </visual>
       <collision>
-        <origin xyz="0 0 0" rpy="1.5708 0 0"/>
-        <geometry>
-          <cylinder radius="${wheel_radius}" length="${wheel_width}"/>
-        </geometry>
+        <origin xyz="${visual_origin}" rpy="${visual_rpy}"/>
+        <geometry><box size="${arm_length} ${arm_thickness} ${arm_depth}"/></geometry>
       </collision>
     </link>
-    <joint name="joint_${name}" type="fixed">
+    <joint name="fix_${name}" type="fixed">
       <parent link="${parent}"/>
-      <child  link="${name}"/>
-      <origin xyz="${x} ${y} ${wheel_origin_z}" rpy="0 0 0"/>
+      <child link="${name}"/>
+      <origin xyz="${x_pos} ${y_pos} 0.000" rpy="0 0 0"/>
     </joint>
   </xacro:macro>
-  <!-- ===================== Instantiate 4 Wheels ===================== -->
-  <!-- Depan = +X, Kiri = +Y -->
-  <xacro:wheel name="wheel_front_left"  parent="base_link" x="${ wheel_x}" y="${ wheel_y}"/>
-  <xacro:wheel name="wheel_front_right" parent="base_link" x="${ wheel_x}" y="${-wheel_y}"/>
-  <xacro:wheel name="wheel_rear_left"   parent="base_link" x="${-wheel_x}" y="${ wheel_y}"/>
-  <xacro:wheel name="wheel_rear_right"  parent="base_link" x="${-wheel_x}" y="${-wheel_y}"/>
+  <!-- WHEEL MACRO -->
+  <xacro:macro name="wheel" params="name parent origin_xyz">
+    <link name="${name}">
+      <visual>
+        <origin xyz="0 0 0" rpy="-1.5708 0 0"/>
+        <geometry><cylinder radius="${wheel_radius}" length="${wheel_width}"/></geometry>
+        <material name="black"/>
+      </visual>
+      <collision>
+        <origin xyz="0 0 0" rpy="-1.5708 0 0"/>
+        <geometry><cylinder radius="${wheel_radius}" length="${wheel_width}"/></geometry>
+      </collision>
+    </link>
+    <joint name="fix_${name}" type="fixed">
+      <parent link="${parent}"/>
+      <child link="${name}"/>
+      <origin xyz="${origin_xyz}" rpy="0 0 0"/>
+    </joint>
+  </xacro:macro>
+  <!-- Instantiate Arms -->
+  <xacro:arm name="arm_front_left" parent="base_link"
+             x_pos="0.200" y_pos="0.520"
+             visual_origin="0.2 -0.230 -0.2" visual_rpy="0 0.785398 0"/>
+  <xacro:arm name="arm_front_right" parent="base_link"
+             x_pos="0.200" y_pos="-0.520"
+             visual_origin="0.2 0.230 -0.2" visual_rpy="0 0.785398 0"/>
+  <xacro:arm name="arm_rear_left" parent="base_link"
+             x_pos="-0.200" y_pos="0.520"
+             visual_origin="-0.2 -0.230 -0.2" visual_rpy="0 0.785398 3.141593"/>
+  <xacro:arm name="arm_rear_right" parent="base_link"
+             x_pos="-0.200" y_pos="-0.520"
+             visual_origin="-0.2 0.230 -0.2" visual_rpy="0 0.785398 3.141593"/>
+  <!-- Instantiate Wheels -->
+  <xacro:wheel name="wheel_front_left" parent="arm_front_left" origin_xyz="0.42426 -0.05 -0.424268"/>
+  <xacro:wheel name="wheel_front_right" parent="arm_front_right" origin_xyz="0.42426 0.05 -0.424268"/>
+  <xacro:wheel name="wheel_rear_left" parent="arm_rear_left" origin_xyz="-0.42426 -0.05 -0.424268"/>
+  <xacro:wheel name="wheel_rear_right" parent="arm_rear_right" origin_xyz="-0.42426 0.05 -0.424268"/>
 </robot>
